File: Keebord.kicad_pcb (KiCad board)
At the start: 2 copper layers, 298 x 100.5 mm, 120 parts, among them SW1 SW_Push, SW10 SW_Push, SW11 SW_Push, SW12 SW_Push, SW13 SW_Push, SW14 SW_Push, SW15 SW_Push, SW16 SW_Push, SW17 SW_Push, SW18 SW_Push, SW19 SW_Push, SW2 SW_Push, SW20 SW_Push, SW21 SW_Push, SW22 SW_Push, SW23 SW_Push, SW24 SW_Push, SW25 SW_Push, SW26 SW_Push, SW27 SW_Push, SW28 SW_Push, SW29 SW_Push, SW3 SW_Push, SW30 SW_Push, SW31 SW_Push, SW32 SW_Push, SW33 SW_Push, SW34 SW_Push, SW35 SW_Push, SW36 SW_Push, SW37 SW_Push, SW38 SW_Push, SW39 SW_Push, SW4 SW_Push, SW40 SW_Push, SW41 SW_Push, SW42 SW_Push, SW43 SW_Push, SW44 SW_Push, SW45 SW_Push, SW46 SW_Push, SW47 SW_Push, SW48 SW_Push, SW49 SW_Push, SW5 SW_Push, SW50 SW_Push, SW51 SW_Push, SW52 SW_Push, SW53 SW_Push, SW54 SW_Push, SW55 SW_Push, SW56 SW_Push, SW57 SW_Push, SW58 SW_Push, SW59 SW_Push, SW6 SW_Push, SW7 SW_Push, SW8 SW_Push, SW9 SW_Push

Commit message: Add files via upload
Parts:
- added JS1: joystick_analog, PCM_marbastlib-xp-various:PNT_psp1000, F.Cu at (287.0, 139.0)
- S1: footprint PCM_marbastlib-mx:STAB_MX_P_6.25u -> PCM_marbastlib-mx:STAB_MX_6u
Connections:
- A1 pad 13: unconnected-(A1-GND-Pad13)_4 -> GND
- A1 pad 18: unconnected-(A1-GND-Pad13)_1 -> GND
- A1 pad 23: unconnected-(A1-GND-Pad13)_6 -> GND
- A1 pad 28: unconnected-(A1-GND-Pad13) -> GND
- A1 pad 3: unconnected-(A1-GND-Pad13)_5 -> GND
- A1 pad 31: unconnected-(A1-GPIO26_ADC0-Pad31) -> Net-(A1-GPIO26_ADC0)
- A1 pad 32: unconnected-(A1-GPIO27_ADC1-Pad32) -> Net-(A1-GPIO27_ADC1)
- A1 pad 36: unconnected-(A1-3V3-Pad36) -> Net-(A1-3V3)
- A1 pad 38: unconnected-(A1-GND-Pad13)_2 -> GND
- A1 pad 8: unconnected-(A1-GND-Pad13)_3 -> GND
Routing:
- net Net-(A1-GPIO26_ADC0): track 0.00 -> 91.4 mm
- net Net-(A1-GPIO27_ADC1): track 0.00 -> 72.1 mm
- net Net-(A1-3V3): track 0.00 -> 71.8 mm
- net GND: track 0.00 -> 44.6 mm, vias 0 -> 1
- added copper zone on F.Cu, net GND
Other:
- board size 298 x 100.5 mm -> 300 x 100 mm
